Commit message: centered the camera by modifying camera.urdf.xacro

File: src/camera_description/urdf/camera.urdf.xacro (robot description, xacro)
@@ -5,4 +5,5 @@
 <xacro:arg name="use_asus_xtion" default="False" />
 <xacro:arg name="camera_pos_z" default="2.0" />
+<xacro:arg name="camera_pos_y" default="-0.0461" />
 <xacro:arg name="camera_pos_x" default="1.0" />
 <xacro:include filename="$(find camera_description)/urdf/camera.gazebo.xacro" />
@@ -14,9 +15,9 @@
    <parent link="camera_footprint" />
    <child link="camera_mount_link" />
-   <origin xyz="0.081 -0.0461 0.15045" rpy="0.0 0.0 ${pi}" />
+   <origin xyz="0.081 ${-0.135+$(arg camera_pos_y)} 0.15045" rpy="0.0 0.0 ${pi}" />
 </joint>
 <link name="camera_mount_link">
    <visual>
-      <origin xyz="${0.00133+$(arg camera_pos_x)} -0.046 ${-0.00326+$(arg camera_pos_z)}" rpy="0.0 ${3*pi/2} 0.0" /> <!--turn -->
+      <origin xyz="${0.00133+$(arg camera_pos_x)} ${0.0+$(arg camera_pos_y)} ${-0.00326+$(arg camera_pos_z)}" rpy="0.0 ${3*pi/2} 0.0" /> <!--turn -->
       <geometry>
          <mesh filename="package://camera_description/meshes/realsense/realsense_mount.stl" scale="0.001 0.001 0.001" />
@@ -25,5 +26,5 @@
    </visual>
    <collision>
-      <origin xyz="${0.00133+$(arg camera_pos_x)} -0.056 ${-0.00326+$(arg camera_pos_z)}" rpy="0.0 ${3*pi/2} 0.0" /> <!--turn -->
+      <origin xyz="${0.00133+$(arg camera_pos_x)} ${-0.01+$(arg camera_pos_y)} ${-0.00326+$(arg camera_pos_z)}" rpy="0.0 ${3*pi/2} 0.0" /> <!--turn -->
       <geometry>
          <box size="0.0175 0.154 0.024" />
@@ -32,5 +33,5 @@
    <inertial>
       <mass value="0.0001" />
-      <origin xyz="0.0000616 -0.0004132 -0.0000000235" />
+      <origin xyz="0.0000616 -0.0004132 -0.0000000235" /> <!--SHOULD I BE CHANGING THIS AS WELL??-->
       <inertia ixx="40.506e-09" ixy="-0.712e-09" ixz="0.472e-09" iyy="2.546e-09" iyz="-0.601e-09" izz="39.799e-09" />
    </inertial>
@@ -38,5 +39,5 @@
 <!-- exectutes the macro in camera_macros.urdf.xacro -->
 <xacro:realsense_camera name="camera" parent="camera_mount_link">
-  <origin xyz="${0.0+$(arg camera_pos_x)} 0.005 ${-0.00337+$(arg camera_pos_z)}" rpy="0.0 ${pi/2} ${pi}" />
+  <origin xyz="${0.0+$(arg camera_pos_x)} ${0.0511+$(arg camera_pos_y)} ${-0.00337+$(arg camera_pos_z)}" rpy="0.0 ${pi/2} ${pi}" />
 </xacro:realsense_camera>
 </xacro:if> <!-- end realsense -->
@@ -45,9 +46,9 @@
    <parent link="camera_footprint" />
    <child link="camera_mount_link" />
-   <origin xyz="0.081 -0.0461 0.15045" rpy="0.0 0.0 ${pi}" />
+   <origin xyz="0.081 ${$(arg camera_pos_y)} 0.15045" rpy="0.0 0.0 ${pi}" />
 </joint>
 <link name="camera_mount_link">
    <visual>
-      <origin xyz="${0.00133+$(arg camera_pos_x)} -0.046 ${-0.00326+$(arg camera_pos_z)}" rpy="0.0 ${3*pi/2} 0.0" />
+      <origin xyz="${0.00133+$(arg camera_pos_x)} ${0.0+$(arg camera_pos_y)} ${-0.00326+$(arg camera_pos_z)}" rpy="0.0 ${3*pi/2} 0.0" />
       <geometry>
          <mesh filename="package://camera_description/meshes/asus_camera/asus_camera_simple.stl" scale="0.001 0.001 0.001" />
@@ -56,5 +57,5 @@
    </visual>
    <collision>
-      <origin xyz="${0.00133+$(arg camera_pos_x)} -0.056 ${-0.00326+$(arg camera_pos_z)}" rpy="0.0 ${3*pi/2} 0.0" />
+      <origin xyz="${0.00133+$(arg camera_pos_x)} ${-0.01+$(arg camera_pos_y)} ${-0.00326+$(arg camera_pos_z)}" rpy="0.0 ${3*pi/2} 0.0" />
       <geometry>
          <box size="0.0175 0.154 0.024" />
@@ -68,5 +69,5 @@
 </link>
 <xacro:asus_camera name="camera" parent="camera_mount_link">
-  <origin xyz="${0.0+$(arg camera_pos_x)} 0.005 ${-0.00337+$(arg camera_pos_z)}" rpy="0.0 ${pi/2} ${pi}" />
+  <origin xyz="${0.0+$(arg camera_pos_x)} ${0.0511+$(arg camera_pos_y)} ${-0.00337+$(arg camera_pos_z)}" rpy="0.0 ${pi/2} ${pi}" />
 </xacro:asus_camera>
 </xacro:if>
